File: trigger.brd (EAGLE design)
At the start: 100 x 29.2 mm, 53 parts, among them IC1 40106N, IC2 78L05Z, T1OUT WQP-PJ301M-12_JACK, T2OUT WQP-PJ301M-12_JACK

Commit message: Minor routing improvement near common output. Added version/date stamp.
Parts:
- moved D5 2.29 mm to (8.89, 12.7), turned to 0 degrees
- moved D4 1.27 mm to (11.4, 17.8)
- moved R23 0.64 mm to (11.4, 22.9)
- turned R14 to 270 degrees
Routing:
- net N$23: track 17.7 -> 12.6 mm
- net N$1: track 14.9 -> 17.8 mm
- net OUT2: track 41.1 -> 42.9 mm, vias 1 -> 0
- net N$21: track 5.61 -> 4.34 mm
- net N$5: track 23.3 -> 23.9 mm
Other:
- board text added: "Gate-to-Trig/Inverter/button module CC BY-SA 2016 Lars Bengtsson v 1.01 20160724"
- board text removed: "Gate-to-Trig/Inverter/button module CC BY-SA 2016 Lars Bengtsson"
